File: Compact Keyboard Schem/Compact Keyboard/Compact Keyboard.kicad_sch (KiCad schematic)
At the start: 7 parts, among them J1 MUX+POT, J2 MUX Power, J4 PAM8406 Power, J6 USB_A, J8 USB_Host

Commit message: Pushing Update
Latest version after PCB printing
Connections:
- net ILI_9341/CS_LCD: now also Teensy_4.1.21 (29); no longer Teensy_4.1.16 (24)
- net ILI_9341/DC_LCD: now also Teensy_4.1.20 (28); no longer Teensy_4.1.17 (25)
- net ILI_9341/LED_LCD: now also Teensy_4.1.17 (25); no longer Teensy_4.1.20 (28)
- net Rotary_Encoder/CLK_RE: now also Teensy_4.1.24 (32); no longer Teensy_4.1.22 (30)
- net Rotary_Encoder/SW_RE: now also Teensy_4.1.22 (30); no longer Teensy_4.1.24 (32)
- net S0_MUX: now also J1.2 (Pin_2); no longer J1.5 (Pin_5)
- net S1_MUX: now also J1.3 (Pin_3); no longer J1.4 (Pin_4)
- net S2_MUX: now also J1.4 (Pin_4); no longer J1.3 (Pin_3)
- net SIG_MUX: now also J1.5 (Pin_5); no longer J1.2 (Pin_2)
