File: Compact Keyboard Schem/Compact Keyboard/ILI9341.kicad_sch (KiCad schematic)
At the start: 4 parts, among them J5 ILI 9341, Q2 Q_PMOS_GSD

Commit message: Pushing Update
Latest version after PCB printing
Parts:
- removed J5: ILI 9341, Connector_PinHeader_2.54mm:PinHeader_1x08_P2.54mm_Vertical, symbol Connector_Generic:Conn_01x08
- added TFT_ILI1: ~, TOMD:ILI9341_TFT, symbol TOMD:ILI9341_TFT
- R6, R7: footprint Resistor_THT:R_Axial_DIN0204_L3.6mm_D1.6mm_P7.62mm_Horizontal -> Resistor_SMD:R_0805_2012Metric_Pad1.20x1.40mm_HandSolder
Connections:
- net +3.3V: now also TFT_ILI1.1 (VCC), TFT_ILI1.4 (RESET)
- net CS_LCD: now also TFT_ILI1.3 (CS)
- net DC_LCD: now also TFT_ILI1.5 (DC)
- net GND: now also TFT_ILI1.2 (GND)
- net MOSI_LCD: now also TFT_ILI1.6 (SDI(MOSI))
- net SCK_LCD: now also TFT_ILI1.7 (SCK)
- net at Q2.3 (D): now also TFT_ILI1.8 (LED)
- no-connect marks 0 -> 10
Changed lines of the file:
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@@
 		(color 0 0 0 0)
+	)
+	(no_connect
+		(at 194.31 114.3)
+	)
+	(no_connect
+		(at 163.83 115.57)
+	)
+	(no_connect
+		(at 194.31 116.84)
+	)
+	(no_connect
+		(at 163.83 125.73)
+	)
+	(no_connect
+		(at 194.31 111.76)
+	)
+	(no_connect
+		(at 163.83 128.27)
+	)
+	(no_connect
+		(at 194.31 109.22)
+	)
+	(no_connect
+		(at 163.83 123.19)
+	)
+	(no_connect
+		(at 163.83 130.81)
+	)
+	(no_connect
+		(at 163.83 120.65)
 	)
 	(wire
@@
 	)
 	(symbol
-		(lib_id "Connector_Generic:Conn_01x08")
-		(at 168.91 102.87 0)
+		(lib_id "TOMD:ILI9341_TFT")
+		(at 179.07 113.03 180)
 		(unit 1)
 		(exclude_from_sim no)
@@
 		(on_board yes)
 		(dnp no)
-		(property "Reference" "J5"
-			(at 168.91 119.38 0)
-			(effects
-				(font
-					(size 1.27 1.27)
-				)
-			)
-		)
-		(property "Value" "ILI 9341"
-			(at 168.91 116.84 0)
-			(effects
-				(font
-					(size 1.27 1.27)
-				)
-			)
-		)
-		(property "Footprint" "Connector_PinHeader_2.54mm:PinHeader_1x08_P2.54mm_Vertical"
-			(at 168.91 102.87 0)
-			(effects
-				(font
-					(size 1.27 1.27)
-				)
-				(hide yes)
-			)
-		)
-		(property "Datasheet" "~"
-			(at 168.91 102.87 0)
-			(effects
-				(font
-					(size 1.27 1.27)
-				)
-				(hide yes)
-			)
-		)
-		(property "Description" "Generic connector, single row, 01x08, script generated (kicad-library-utils/schlib/autogen/connector/)"
-			(at 168.91 102.87 0)
-			(effects
-				(font
-					(size 1.27 1.27)
-				)
-				(hide yes)
-			)
+		(fields_autoplaced yes)
+		(property "Reference" "TFT_ILI1"
+			(at 179.07 87.63 0)
+			(effects
+				(font
+					(size 1.27 1.27)
+				)
+			)
+		)
+		(property "Value" "~"
+			(at 179.07 90.17 0)
+			(effects
+				(font
+					(size 1.27 1.27)
+				)
+			)
+		)
+		(property "Footprint" "TOMD:ILI9341_TFT"
+			(at 179.07 113.03 0)
+			(effects
+				(font
+					(size 1.27 1.27)
+				)
+				(hide yes)
+			)
+		)
+		(property "Datasheet" ""
+			(at 179.07 113.03 0)
+			(effects
+				(font
+					(size 1.27 1.27)
+				)
+				(hide yes)
+			)
+		)
+		(property "Description" ""
+			(at 179.07 113.03 0)
+			(effects
+				(font
+					(size 1.27 1.27)
+				)
+				(hide yes)
+			)
+		)
+		(pin "15"
+		)
+		(pin "5"
+		)
+		(pin "4"
+		)
+		(pin "16"
+		)
+		(pin "9"
+		)
+		(pin "17"
+		)
+		(pin "11"
+		)
+		(pin "3"
+		)
+		(pin "14"
+		)
+		(pin "13"
+		)
+		(pin "18"
 		)
 		(pin "8"
 		)
+		(pin "6"
+		)
+		(pin "12"
+		)
+		(pin "10"
+		)
 		(pin "7"
 		)
+		(pin "2"
+		)
 		(pin "1"
 		)
-		(pin "2"
-		)
-		(pin "5"
-		)
-		(pin "4"
-		)
-		(pin "3"
-		)
-		(pin "6"
-		)
 		(instances
-			(project "Compact Keyboard"
+			(project ""
 				(path "/ab0b387f-d15a-4769-b7a7-126c2f26f021/75defc31-3db0-4477-a55a-5e4fcab5c387"
-					(reference "J5")
+					(reference "TFT_ILI1")
 					(unit 1)
 				)
@@
 			)
 		)
-		(property "Footprint" "Resistor_THT:R_Axial_DIN0204_L3.6mm_D1.6mm_P7.62mm_Horizontal"
+		(property "Footprint" "Resistor_SMD:R_0805_2012Metric_Pad1.20x1.40mm_HandSolder"
 			(at 127 133.858 90)
 			(effects
@@
 			)
 		)
-		(property "Footprint" "Resistor_THT:R_Axial_DIN0204_L3.6mm_D1.6mm_P7.62mm_Horizontal"
+		(property "Footprint" "Resistor_SMD:R_0805_2012Metric_Pad1.20x1.40mm_HandSolder"
 			(at 127 124.968 90)
 			(effects
