File: Compact Keyboard Schem/Compact Keyboard/RotaryEncoder.kicad_sch (KiCad schematic)
At the start: 3 parts, among them J7 Rotary_Encoder

Commit message: Pushing Update
Latest version after PCB printing
Parts:
- removed J7: Rotary_Encoder, Connector_PinHeader_2.54mm:PinHeader_1x05_P2.54mm_Horizontal, symbol Connector_Generic:Conn_01x05
- added R10, R8, R9: 10K, Resistor_SMD:R_0805_2012Metric_Pad1.20x1.40mm_HandSolder, symbol Device:R
- added SW1: RotaryEncoder_Switch_MP, Rotary_Encoder:RotaryEncoder_Alps_EC11E-Switch_Vertical_H20mm, symbol Device:RotaryEncoder_Switch_MP
Connections:
- net +3.3V: now also R10.2, R8.1, R9.1
- net CLK_RE: now also R9.2, SW1.B
- net DT_RE: now also R8.2, SW1.A
- net GND: now also SW1.C, SW1.MP, SW1.S2
- net SW_RE: now also R10.1, SW1.S1
