File: Compact Keyboard Schem/Compact Keyboard/powerProtection.kicad_sch (KiCad schematic)
At the start: 6 parts, among them J9 Jack-DC, Q1 Q_PMOS_GSD, SW1 SW_Push_LED

Commit message: Pushing Update
Latest version after PCB printing
Parts:
- removed Q1: Q_PMOS_GSD, Package_TO_SOT_SMD:SOT-23, symbol Transistor_FET:Q_PMOS_GSD
- removed SW1: SW_Push_LED, Connector_Wire:SolderWire-0.25sqmm_1x04_P4.2mm_D0.65mm_OD1.7mm_Relief, symbol Switch:SW_Push_LED
- added J3: SW_Switch_LED, Connector_Wire:SolderWire-0.25sqmm_1x04_P4.2mm_D0.65mm_OD1.7mm_Relief, symbol Connector_Generic:Conn_01x04
- added Q3: Q_PMOS_GDS, Package_TO_SOT_THT:TO-220F-3_Vertical, symbol Transistor_FET:Q_PMOS_GDS
- R1: footprint Resistor_THT:R_Axial_DIN0204_L3.6mm_D1.6mm_P7.62mm_Horizontal -> Resistor_SMD:R_0805_2012Metric_Pad1.20x1.40mm_HandSolder
Connections:
- net +5V: now also Q3.2 (D)
- net GND: now also J3.3 (Pin_3), Q3.1 (G)
- net at J9.1, R1.2: now also J3.1 (Pin_1)
- net at R1.1: now also J3.2 (Pin_2)
- new net: J3.4 (Pin_4), Q3.3 (S)
Other:
- moved on the sheet: R1
