File: Compact Keyboard Schem/Potentiometer+MUX/Potentiometer+MUX.kicad_sch (KiCad schematic)
At the start: 14 parts, among them J1 Conn_01x04, J2 Conn_01x02, J3 Conn_01x08, J4 Conn_01x16

Commit message: Pushing Update
Latest version after PCB printing
Parts:
- renumbered C9 to C1
Connections:
- net GND: now also J3.7 (Pin_7)
- no-connect marks 18 -> 16
Changed lines of the file:
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@@
+	)
+	(junction
+		(at 165.1 102.87)
+		(diameter 0)
+		(color 0 0 0 0)
 	)
 	(junction
@@
 	(junction
 		(at 203.2 104.14)
+		(diameter 0)
+		(color 0 0 0 0)
+	)
+	(junction
+		(at 175.26 102.87)
 		(diameter 0)
 		(color 0 0 0 0)
@@
 	)
 	(no_connect
-		(at 162.56 86.36)
-	)
-	(no_connect
 		(at 147.32 106.68)
 	)
@@
 	)
 	(no_connect
-		(at 163.83 35.56)
-	)
-	(no_connect
 		(at 147.32 101.6)
 	)
@@
 	(wire
 		(pts
-			(xy 167.64 102.87) (xy 195.58 102.87)
+			(xy 167.64 102.87) (xy 175.26 102.87)
 		)
 		(stroke
@@
 	(wire
 		(pts
+			(xy 175.26 35.56) (xy 175.26 102.87)
+		)
+		(stroke
+			(width 0)
+			(type default)
+		)
+	)
+	(wire
+		(pts
 			(xy 55.88 69.85) (xy 66.04 69.85)
 		)
@@
 	(wire
 		(pts
-			(xy 162.56 102.87) (xy 167.64 102.87)
+			(xy 162.56 102.87) (xy 165.1 102.87)
 		)
 		(stroke
@@
 	(wire
 		(pts
+			(xy 165.1 102.87) (xy 167.64 102.87)
+		)
+		(stroke
+			(width 0)
+			(type default)
+		)
+	)
+	(wire
+		(pts
 			(xy 162.56 93.98) (xy 172.72 93.98)
 		)
@@
 	(wire
 		(pts
+			(xy 175.26 102.87) (xy 195.58 102.87)
+		)
+		(stroke
+			(width 0)
+			(type default)
+		)
+	)
+	(wire
+		(pts
 			(xy 62.23 119.38) (xy 62.23 133.35)
 		)
@@
 	(wire
 		(pts
+			(xy 162.56 86.36) (xy 165.1 86.36)
+		)
+		(stroke
+			(width 0)
+			(type default)
+		)
+	)
+	(wire
+		(pts
 			(xy 212.09 102.87) (xy 212.09 104.14)
 		)
@@
 	(wire
 		(pts
+			(xy 165.1 86.36) (xy 165.1 102.87)
+		)
+		(stroke
+			(width 0)
+			(type default)
+		)
+	)
+	(wire
+		(pts
 			(xy 203.2 99.06) (xy 170.18 99.06)
+		)
+		(stroke
+			(width 0)
+			(type default)
+		)
+	)
+	(wire
+		(pts
+			(xy 163.83 35.56) (xy 175.26 35.56)
 		)
 		(stroke
@@
 		(dnp no)
 		(fields_autoplaced yes)
-		(property "Reference" "C9"
+		(property "Reference" "C1"
 			(at 205.74 100.3362 0)
 			(effects
@@
 			(project ""
 				(path "/78e67f7c-5e13-4d41-8b0c-90d89c59b709"
-					(reference "C9")
+					(reference "C1")
 					(unit 1)
 				)
